File: Arduino_LCD.kicad_pcb (KiCad board)
At the start: 2 copper layers, 68.6 x 53.3 mm, 40 parts, among them J1 Conn_02x07_Odd_Even, J2 Vsens, J3 Isense, J4 DPsense, J5 Psense, P1 Power, P2 Analog, P3 Digital, P4 Digital, P5 CONN_01X01, P6 CONN_01X01, P7 CONN_01X01, P8 CONN_01X01, Q1 Q_NPN_EBC, Q2 Q_NPN_EBC, U1 LM324, U2 AMS1117, U2 AP2112K-3.3, U3 ESP-01v090

Commit message: added
Parts:
- removed the U2 at (166.1, 145.1)
- moved C3 104.9 mm to (118.9, 111.9), turned to 180 degrees
- moved R7 98.5 mm to (146.5, 85.5), turned to 90 degrees
- moved R11 90.5 mm to (146.5, 98.1), turned to 270 degrees
- moved RV1 89.5 mm to (117.3, 100.8), turned to 90 degrees
- moved C5 84.3 mm to (144.4, 98.2), turned to 270 degrees
- moved U2 83.6 mm to (129.0, 106.7)
- moved C4 82.4 mm to (161.0, 84.3), turned to 90 degrees
- moved Q2 72.5 mm to (140.8, 104.1), turned to 270 degrees
- moved Q1 70.2 mm to (134.5, 106.1)
- moved R2 58.2 mm to (133.9, 101.2)
- moved C2 56.5 mm to (125.5, 106.7), turned to 90 degrees
- moved J1 54.4 mm to (126.1, 96.6), turned to 180 degrees
- moved R4 51.0 mm to (138.6, 112.1)
- moved C1 50.4 mm to (129.0, 109.7)
- moved R3 45.3 mm to (142.2, 109.6), turned to 180 degrees
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Connections:
- J1 pad 10: (no net) -> Net-(J1-Pad10)
- J1 pad 7: (no net) -> Net-(J1-Pad7)
- J1 pad 8: (no net) -> Net-(J1-Pad8)
- J1 pad 9: (no net) -> Net-(J1-Pad9)
- P1 pad 1: (no net) -> Net-(P1-Pad1)
- P1 pad 2: (no net) -> /IOREF
- P1 pad 3: (no net) -> /Reset
- P3 pad 3: (no net) -> /AREF
- P4 pad 1: (no net) -> /7
- P4 pad 2: (no net) -> /6(**)
- P4 pad 7: (no net) -> /1(Tx)
- P4 pad 8: (no net) -> /0(Rx)
- P5 pad 1: (no net) -> Net-(P5-Pad1)
- P6 pad 1: (no net) -> Net-(P6-Pad1)
- P7 pad 1: (no net) -> Net-(P7-Pad1)
- P8 pad 1: (no net) -> Net-(P8-Pad1)
- U2 pad 4: (no net) -> Net-(U2-Pad4)
- U3 pad 4: (no net) -> Net-(U3-Pad4)
Routing:
- net /2: track 0.00 -> 64.9 mm
- net /Vin: track 0.00 -> 62.8 mm, vias 0 -> 2
- net /3(**): track 0.00 -> 61.1 mm
- net /4: track 0.00 -> 52.1 mm
- net /A0: track 0.00 -> 49.5 mm, vias 0 -> 3
- net /5(**): track 0.00 -> 39.9 mm, vias 0 -> 1
- net /A1: track 0.00 -> 36.7 mm, vias 0 -> 1
- net Net-(J2-Pad1): track 0.00 -> 35.7 mm, vias 0 -> 1
- net /8: track 0.00 -> 31.7 mm
- net GND: track 0.00 -> 31.0 mm, vias 0 -> 2
- net /9(**): track 0.00 -> 28.1 mm
- net /10(**_SS): track 0.00 -> 25.9 mm
- net /A3: track 0.00 -> 24.7 mm, vias 0 -> 1
- net Net-(J3-Pad1): track 0.00 -> 24.1 mm
- net Net-(C5-Pad1): track 0.00 -> 20.4 mm
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- added copper zone on F.Cu, net +3V3
- added copper zone on F.Cu, net +5V
- added copper zone on B.Cu, net GND
Other:
- rule trace_min: 0.2 -> 0.1524
- rule via_min_drill: 0.3 -> 0.254
- rule via_min_size: 0.4 -> 0.508
