File: Arduino_LCD.sch (KiCad schematic (older format))
At the start: 39 parts, among them J1 Conn_02x07_Odd_Even, J2 Vsens, J3 Isense, J4 DPsense, J5 Psense, P1 Power, P2 Analog, P3 Digital, P4 Digital, P5 CONN_01X01, P6 CONN_01X01, P7 CONN_01X01, P8 CONN_01X01, Q1 Q_NPN_EBC, Q2 Q_NPN_EBC, U1 LM324, U2 AP2112K-3.3, U3 ESP-01v090

Commit message: added
Parts:
- U3: symbol ESP_8266:ESP-01v090 -> Arduino_LCD-rescue:ESP-01v090-ESP_8266
Changed lines of the file:
@@
 Connection ~ 8900 4750
 $Comp
-L ESP_8266:ESP-01v090 U3
+L Arduino_LCD-rescue:ESP-01v090-ESP_8266 U3
 U 1 1 5EAB519A
 P 6450 2650
